File: KiCad/GripCtrl.kicad_sch (KiCad schematic)
At the start: 18 parts, among them SW1 SW_Push, SW10 SW_Push, SW11 SW_Push, SW2 SW_Push, SW3 SW_Push, SW4 SW_Push, SW5 SW_Push, SW6 SW_Push, SW7 SW_Push, SW8 SW_Push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

Commit message: Update schematic
Other:
- note added: "Receiver Only"
- moved on the sheet: BZZR1, FF01 E-STOP1, JYSTK1, JYSTK2, SSD1

Commit message: Add title to schematic
Other:
- title: (none) -> GripCtrl - Unified Wiring Diagram
Changed lines of the file:
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@@
 	(generator_version "9.0")
 	(paper "A4")
+	(title_block
+		(title "GripCtrl - Unified Wiring Diagram")
+	)
 	(rectangle
 		(start 194.31 35.56)
